File: F0-uConsole.kicad_sch (KiCad schematic)
At the start: 5 parts, among them J1 uConsoleEXT, J2 F0_1, J3 F0_2, J4 USB1, J5 USB2

Commit message: Upload Rev0.2 board
change notes: 
added speaker terminals
flipped the flipper connector so the module face would be facing the user. basically this meant a full redesign.
shortened the card slightly.
Parts:
- added J6 (x2): uConsoleSpeaker, @upico:speaker, symbol @upico:uConsoleSpeaker
Connections:
- net SPK_LP: now reaches J1.1 (SPK_LP)
- net SPK_LP: now also J6.1 (P1), J6.3 (P2)
- net SPK_RP: now reaches J1.14 (SPK_RP)
- net SPK_RP: now also J6.1 (P1), J6.3 (P2)
- net SKP_RN: now reaches J1.16 (SPK_RN)
- net SKP_RN: now also J6.2 (N1), J6.4 (N2)
- net SKP_LN: now reaches J1.3 (SPK_LN)
- net SKP_LN: now also J6.2 (N1), J6.4 (N2)
